Commit message: added my_robot_bringup package for gazebo simulation
Signed-off-by: Albert <wensinlor@gmail.com>

File: install/my_robot_description/share/my_robot_description/urdf/common_properties.xacro (robot description, xacro)
@@ -7,3 +7,30 @@
         <color rgba="0.5 0.5 0.5 1"/>
     </material>
+    <xacro:macro name="box_inertia" params="m l w h xyz rpy">
+        <intertial>
+            <origin xyz="${xyz}" rpy="${rpy}"/>
+            <mass value="${m}"/>
+            <inertia ixx="${(m/12) * (h*h + l*l)}" ixy="0" ixz="0"
+                     iyy="${(m/12) * (w*w + l*l)}" iyz="0"
+                     izz="${(m/12) * (w*w + h*h)}"/>
+        </intertial>
+    </xacro:macro>
+    <xacro:macro name="cylinder_inertia" params="m r h xyz rpy">
+        <intertial>
+            <origin xyz="${xyz}" rpy="${rpy}"/>
+            <mass value="${m}"/>
+            <inertia ixx="${(m/12) * (3*r*r + h*h)}" ixy="0" ixz="0"
+                     iyy="${(m/12) * (3*r*r + h*h)}" iyz="0"
+                     izz="${(m/2) * (r*r)}"/>
+        </intertial>
+    </xacro:macro>
+    <xacro:macro name="sphere_inertia" params="m r xyz rpy">
+        <intertial>
+            <origin xyz="${xyz}" rpy="${rpy}"/>
+            <mass value="${m}"/>
+            <inertia ixx="${(2/5)*m*r*r}" ixy="0" ixz="0"
+                     iyy="${(2/5)*m*r*r}" iyz="0"
+                     izz="${(2/5)*m*r*r}"/>
+        </intertial>
+    </xacro:macro>
 </robot>

File: install/my_robot_description/share/my_robot_description/urdf/mobile_base.xacro (robot description, xacro)
@@ -15,4 +15,12 @@
             <material name="blue"/>
         </visual>
+        <collision>
+            <geometry>
+                <box size="${base_length} ${base_width} ${base_height}"/>
+            </geometry>
+            <origin xyz="0 0 ${base_height / 2.0}" rpy="0 0 0"/>
+        </collision>
+        <xacro:box_inertia m="5.0" l="${base_length}" w="${base_width}" h="${base_height}"
+                           xyz="0 0 ${base_height / 2.0}" rpy="0 0 0"/>
     </link>
     <xacro:macro name="wheel_link" params="prefix">
@@ -25,4 +33,12 @@
                 <material name="grey"/>
             </visual>
+            <collision>
+                <geometry>
+                    <cylinder radius="${wheel_radius}" length="${wheel_length}"/>
+                </geometry>
+                <origin xyz="0 0 0" rpy="${pi / 2.0} 0 0"/>
+            </collision>
+            <xacro:cylinder_inertia m="1.0" r="${wheel_radius}" h="${wheel_length}"
+                                    xyz="0 0 0" rpy="${pi / 2.0} 0 0"/>
         </link>
     </xacro:macro>
@@ -55,4 +71,12 @@
             <material name="grey"/>
         </visual>
+        <collision>
+            <geometry>
+                <sphere radius="${wheel_radius / 2.0}"/>
+            </geometry>
+            <origin xyz="0 0 0" rpy="0 0 0"/>
+        </collision>
+        <xacro:sphere_inertia m="0.5" r="${wheel_radius / 2.0}"
+                              xyz="0 0 0" rpy="0 0 0"/>
     </link>
     <joint name="base_joint" type="fixed">

Commit message: create world in gazebo and added sensor to the robot
Signed-off-by: Albert <wensinlor@gmail.com>

File: install/my_robot_description/share/my_robot_description/urdf/common_properties.xacro (robot description, xacro)
@@ -8,5 +8,5 @@
     </material>
     <xacro:macro name="box_inertia" params="m l w h xyz rpy">
-        <intertial>
+        <inertial>
             <origin xyz="${xyz}" rpy="${rpy}"/>
             <mass value="${m}"/>
@@ -14,8 +14,8 @@
                      iyy="${(m/12) * (w*w + l*l)}" iyz="0"
                      izz="${(m/12) * (w*w + h*h)}"/>
-        </intertial>
+        </inertial>
     </xacro:macro>
     <xacro:macro name="cylinder_inertia" params="m r h xyz rpy">
-        <intertial>
+        <inertial>
             <origin xyz="${xyz}" rpy="${rpy}"/>
             <mass value="${m}"/>
@@ -23,8 +23,8 @@
                      iyy="${(m/12) * (3*r*r + h*h)}" iyz="0"
                      izz="${(m/2) * (r*r)}"/>
-        </intertial>
+        </inertial>
     </xacro:macro>
     <xacro:macro name="sphere_inertia" params="m r xyz rpy">
-        <intertial>
+        <inertial>
             <origin xyz="${xyz}" rpy="${rpy}"/>
             <mass value="${m}"/>
@@ -32,5 +32,5 @@
                      iyy="${(2/5)*m*r*r}" iyz="0"
                      izz="${(2/5)*m*r*r}"/>
-        </intertial>
+        </inertial>
     </xacro:macro>
 </robot>

File: install/my_robot_description/share/my_robot_description/urdf/my_robot.urdf.xacro (robot description, xacro)
@@ -1,6 +1,7 @@
 <?xml version="1.0"?>
 <robot name="my_robot" xmlns:xacro="http://www.ros.org/wiki/xacro">
-    <xacro:include filename="common_properties.xacro"/>
-    <xacro:include filename="mobile_base.xacro"/>
-    <xacro:include filename="mobile_base_gazebo.xacro"/>
+    <xacro:include filename="common_properties.xacro" />
+    <xacro:include filename="mobile_base.xacro" />
+    <xacro:include filename="mobile_base_gazebo.xacro" />
+    <xacro:include filename="camera.xacro"/>
 </robot>

Commit message: finished final project
Signed-off-by: Albert <wensinlor@gmail.com>

File: install/my_robot_description/share/my_robot_description/urdf/common_properties.xacro (robot description, xacro)
@@ -6,4 +6,10 @@
     <material name="grey">
         <color rgba="0.5 0.5 0.5 1"/>
+    </material>
+    <material name="orange">
+        <color rgba="1.0 0.5 0 1"/>
+    </material>
+    <material name="yellow">
+        <color rgba="1.0 1.0 0 1"/>
     </material>
     <xacro:macro name="box_inertia" params="m l w h xyz rpy">

File: install/my_robot_description/share/my_robot_description/urdf/my_robot.urdf.xacro (robot description, xacro)
@@ -4,4 +4,11 @@
     <xacro:include filename="mobile_base.xacro" />
     <xacro:include filename="mobile_base_gazebo.xacro" />
+    <xacro:include filename="arm.xacro" />
+    <xacro:include filename="arm_gazebo.xacro" />
+    <joint name="mobile_base_arm_joint" type="fixed">
+        <parent link="base_link"/>
+        <child link="arm_base_link"/>
+        <origin xyz="${base_length / 4.0} 0 ${base_height}" rpy="0 0 0"/>
+    </joint>
     <xacro:include filename="camera.xacro"/>
 </robot>
